Commit message: Update README and remove redundant "_mesh" suffix

File: urdf/jaxon_jvrc.urdf (robot description, URDF)
Before this commit: robot JAXON_JVRC, 39 links, 38 joints
Links:
- link BODY: geometry collision mesh filename=../meshes/BODY.dae scale=1 1 1; visual mesh filename=../meshes/BODY.dae scale=1 1 1
- link CHEST_LINK0: geometry collision mesh filename=../meshes/CHEST_LINK0.dae scale=1 1 1; visual mesh filename=../meshes/CHEST_LINK0.dae scale=1 1 1
- link CHEST_LINK1: geometry collision mesh filename=../meshes/CHEST_LINK1.dae scale=1 1 1; visual mesh filename=../meshes/CHEST_LINK1.dae scale=1 1 1
- link CHEST_LINK2: geometry collision mesh filename=../meshes/CHEST_LINK2.dae scale=1 1 1; visual mesh filename=../meshes/CHEST_LINK2.dae scale=1 1 1
- link HEAD_LINK0: geometry collision mesh filename=../meshes/HEAD_LINK0.dae scale=1 1 1; visual mesh filename=../meshes/HEAD_LINK0.dae scale=1 1 1
- link HEAD_LINK1: geometry collision mesh filename=../meshes/HEAD_LINK1.dae scale=1 1 1; visual mesh filename=../meshes/HEAD_LINK1.dae scale=1 1 1
- link LARM_FINGER0: geometry collision mesh filename=../meshes/LARM_FINGER0.dae scale=1 1 1; visual mesh filename=../meshes/LARM_FINGER0.dae scale=1 1 1
- link LARM_FINGER1: geometry collision mesh filename=../meshes/LARM_FINGER1.dae scale=1 1 1; visual mesh filename=../meshes/LARM_FINGER1.dae scale=1 1 1
- link LARM_LINK0: geometry collision mesh filename=../meshes/LARM_LINK0.dae scale=1 1 1; visual mesh filename=../meshes/LARM_LINK0.dae scale=1 1 1
- link LARM_LINK1: geometry collision mesh filename=../meshes/LARM_LINK1.dae scale=1 1 1; visual mesh filename=../meshes/LARM_LINK1.dae scale=1 1 1
- link LARM_LINK2: geometry collision mesh filename=../meshes/LARM_LINK2.dae scale=1 1 1; visual mesh filename=../meshes/LARM_LINK2.dae scale=1 1 1
- link LARM_LINK3: geometry collision mesh filename=../meshes/LARM_LINK3.dae scale=1 1 1; visual mesh filename=../meshes/LARM_LINK3.dae scale=1 1 1
- link LARM_LINK4: geometry collision mesh filename=../meshes/LARM_LINK4.dae scale=1 1 1; visual mesh filename=../meshes/LARM_LINK4.dae scale=1 1 1
- link LARM_LINK5: geometry collision mesh filename=../meshes/LARM_LINK5.dae scale=1 1 1; visual mesh filename=../meshes/LARM_LINK5.dae scale=1 1 1
- link LARM_LINK6: geometry collision mesh filename=../meshes/LARM_LINK6.dae scale=1 1 1; visual mesh filename=../meshes/LARM_LINK6.dae scale=1 1 1
- link LARM_LINK7: geometry collision mesh filename=../meshes/LARM_LINK7.dae scale=1 1 1; visual mesh filename=../meshes/LARM_LINK7.dae scale=1 1 1
- link LLEG_LINK0: geometry collision mesh filename=../meshes/LLEG_LINK0.dae scale=1 1 1; visual mesh filename=../meshes/LLEG_LINK0.dae scale=1 1 1
- link LLEG_LINK1: geometry collision mesh filename=../meshes/LLEG_LINK1.dae scale=1 1 1; visual mesh filename=../meshes/LLEG_LINK1.dae scale=1 1 1
- link LLEG_LINK2: geometry collision mesh filename=../meshes/LLEG_LINK2.dae scale=1 1 1; visual mesh filename=../meshes/LLEG_LINK2.dae scale=1 1 1
- link LLEG_LINK3: geometry collision mesh filename=../meshes/LLEG_LINK3.dae scale=1 1 1; visual mesh filename=../meshes/LLEG_LINK3.dae scale=1 1 1
- link LLEG_LINK4: geometry collision mesh filename=../meshes/LLEG_LINK4.dae scale=1 1 1; visual mesh filename=../meshes/LLEG_LINK4.dae scale=1 1 1
- link LLEG_LINK5: geometry collision mesh filename=../meshes/LLEG_LINK5.dae scale=1 1 1; visual mesh filename=../meshes/LLEG_LINK5.dae scale=1 1 1
- link RANGE_LINK: geometry collision mesh filename=../meshes/RANGE_LINK.dae scale=1 1 1; visual mesh filename=../meshes/RANGE_LINK.dae scale=1 1 1
- link RARM_FINGER0: geometry collision mesh filename=../meshes/RARM_FINGER0.dae scale=1 1 1; visual mesh filename=../meshes/RARM_FINGER0.dae scale=1 1 1
- link RARM_FINGER1: geometry collision mesh filename=../meshes/RARM_FINGER1.dae scale=1 1 1; visual mesh filename=../meshes/RARM_FINGER1.dae scale=1 1 1
- link RARM_LINK0: geometry collision mesh filename=../meshes/RARM_LINK0.dae scale=1 1 1; visual mesh filename=../meshes/RARM_LINK0.dae scale=1 1 1
- link RARM_LINK1: geometry collision mesh filename=../meshes/RARM_LINK1.dae scale=1 1 1; visual mesh filename=../meshes/RARM_LINK1.dae scale=1 1 1
- link RARM_LINK2: geometry collision mesh filename=../meshes/RARM_LINK2.dae scale=1 1 1; visual mesh filename=../meshes/RARM_LINK2.dae scale=1 1 1
- link RARM_LINK3: geometry collision mesh filename=../meshes/RARM_LINK3.dae scale=1 1 1; visual mesh filename=../meshes/RARM_LINK3.dae scale=1 1 1
- link RARM_LINK4: geometry collision mesh filename=../meshes/RARM_LINK4.dae scale=1 1 1; visual mesh filename=../meshes/RARM_LINK4.dae scale=1 1 1
- link RARM_LINK5: geometry collision mesh filename=../meshes/RARM_LINK5.dae scale=1 1 1; visual mesh filename=../meshes/RARM_LINK5.dae scale=1 1 1
- link RARM_LINK6: geometry collision mesh filename=../meshes/RARM_LINK6.dae scale=1 1 1; visual mesh filename=../meshes/RARM_LINK6.dae scale=1 1 1
- link RARM_LINK7: geometry collision mesh filename=../meshes/RARM_LINK7.dae scale=1 1 1; visual mesh filename=../meshes/RARM_LINK7.dae scale=1 1 1
- link RLEG_LINK0: geometry collision mesh filename=../meshes/RLEG_LINK0.dae scale=1 1 1; visual mesh filename=../meshes/RLEG_LINK0.dae scale=1 1 1
- link RLEG_LINK1: geometry collision mesh filename=../meshes/RLEG_LINK1.dae scale=1 1 1; visual mesh filename=../meshes/RLEG_LINK1.dae scale=1 1 1
- link RLEG_LINK2: geometry collision mesh filename=../meshes/RLEG_LINK2.dae scale=1 1 1; visual mesh filename=../meshes/RLEG_LINK2.dae scale=1 1 1
- link RLEG_LINK3: geometry collision mesh filename=../meshes/RLEG_LINK3.dae scale=1 1 1; visual mesh filename=../meshes/RLEG_LINK3.dae scale=1 1 1
- link RLEG_LINK4: geometry collision mesh filename=../meshes/RLEG_LINK4.dae scale=1 1 1; visual mesh filename=../meshes/RLEG_LINK4.dae scale=1 1 1
- link RLEG_LINK5: geometry collision mesh filename=../meshes/RLEG_LINK5.dae scale=1 1 1; visual mesh filename=../meshes/RLEG_LINK5.dae scale=1 1 1

Commit message: Update relative paths to package:// paths

File: urdf/jaxon_jvrc.urdf (robot description, URDF)
Before this commit: robot JAXON_JVRC, 39 links, 38 joints
Links:
- link BODY: geometry collision mesh filename=package://jaxon_description/BODY.dae scale=1 1 1; visual mesh filename=package://jaxon_description/BODY.dae scale=1 1 1
- link CHEST_LINK0: geometry collision mesh filename=package://jaxon_description/CHEST_LINK0.dae scale=1 1 1; visual mesh filename=package://jaxon_description/CHEST_LINK0.dae scale=1 1 1
- link CHEST_LINK1: geometry collision mesh filename=package://jaxon_description/CHEST_LINK1.dae scale=1 1 1; visual mesh filename=package://jaxon_description/CHEST_LINK1.dae scale=1 1 1
- link CHEST_LINK2: geometry collision mesh filename=package://jaxon_description/CHEST_LINK2.dae scale=1 1 1; visual mesh filename=package://jaxon_description/CHEST_LINK2.dae scale=1 1 1
- link HEAD_LINK0: geometry collision mesh filename=package://jaxon_description/HEAD_LINK0.dae scale=1 1 1; visual mesh filename=package://jaxon_description/HEAD_LINK0.dae scale=1 1 1
- link HEAD_LINK1: geometry collision mesh filename=package://jaxon_description/HEAD_LINK1.dae scale=1 1 1; visual mesh filename=package://jaxon_description/HEAD_LINK1.dae scale=1 1 1
- link LARM_FINGER0: geometry collision mesh filename=package://jaxon_description/LARM_FINGER0.dae scale=1 1 1; visual mesh filename=package://jaxon_description/LARM_FINGER0.dae scale=1 1 1
- link LARM_FINGER1: geometry collision mesh filename=package://jaxon_description/LARM_FINGER1.dae scale=1 1 1; visual mesh filename=package://jaxon_description/LARM_FINGER1.dae scale=1 1 1
- link LARM_LINK0: geometry collision mesh filename=package://jaxon_description/LARM_LINK0.dae scale=1 1 1; visual mesh filename=package://jaxon_description/LARM_LINK0.dae scale=1 1 1
- link LARM_LINK1: geometry collision mesh filename=package://jaxon_description/LARM_LINK1.dae scale=1 1 1; visual mesh filename=package://jaxon_description/LARM_LINK1.dae scale=1 1 1
- link LARM_LINK2: geometry collision mesh filename=package://jaxon_description/LARM_LINK2.dae scale=1 1 1; visual mesh filename=package://jaxon_description/LARM_LINK2.dae scale=1 1 1
- link LARM_LINK3: geometry collision mesh filename=package://jaxon_description/LARM_LINK3.dae scale=1 1 1; visual mesh filename=package://jaxon_description/LARM_LINK3.dae scale=1 1 1
- link LARM_LINK4: geometry collision mesh filename=package://jaxon_description/LARM_LINK4.dae scale=1 1 1; visual mesh filename=package://jaxon_description/LARM_LINK4.dae scale=1 1 1
- link LARM_LINK5: geometry collision mesh filename=package://jaxon_description/LARM_LINK5.dae scale=1 1 1; visual mesh filename=package://jaxon_description/LARM_LINK5.dae scale=1 1 1
- link LARM_LINK6: geometry collision mesh filename=package://jaxon_description/LARM_LINK6.dae scale=1 1 1; visual mesh filename=package://jaxon_description/LARM_LINK6.dae scale=1 1 1
- link LARM_LINK7: geometry collision mesh filename=package://jaxon_description/LARM_LINK7.dae scale=1 1 1; visual mesh filename=package://jaxon_description/LARM_LINK7.dae scale=1 1 1
- link LLEG_LINK0: geometry collision mesh filename=package://jaxon_description/LLEG_LINK0.dae scale=1 1 1; visual mesh filename=package://jaxon_description/LLEG_LINK0.dae scale=1 1 1
- link LLEG_LINK1: geometry collision mesh filename=package://jaxon_description/LLEG_LINK1.dae scale=1 1 1; visual mesh filename=package://jaxon_description/LLEG_LINK1.dae scale=1 1 1
- link LLEG_LINK2: geometry collision mesh filename=package://jaxon_description/LLEG_LINK2.dae scale=1 1 1; visual mesh filename=package://jaxon_description/LLEG_LINK2.dae scale=1 1 1
- link LLEG_LINK3: geometry collision mesh filename=package://jaxon_description/LLEG_LINK3.dae scale=1 1 1; visual mesh filename=package://jaxon_description/LLEG_LINK3.dae scale=1 1 1
- link LLEG_LINK4: geometry collision mesh filename=package://jaxon_description/LLEG_LINK4.dae scale=1 1 1; visual mesh filename=package://jaxon_description/LLEG_LINK4.dae scale=1 1 1
- link LLEG_LINK5: geometry collision mesh filename=package://jaxon_description/LLEG_LINK5.dae scale=1 1 1; visual mesh filename=package://jaxon_description/LLEG_LINK5.dae scale=1 1 1
- link RANGE_LINK: geometry collision mesh filename=package://jaxon_description/RANGE_LINK.dae scale=1 1 1; visual mesh filename=package://jaxon_description/RANGE_LINK.dae scale=1 1 1
- link RARM_FINGER0: geometry collision mesh filename=package://jaxon_description/RARM_FINGER0.dae scale=1 1 1; visual mesh filename=package://jaxon_description/RARM_FINGER0.dae scale=1 1 1
- link RARM_FINGER1: geometry collision mesh filename=package://jaxon_description/RARM_FINGER1.dae scale=1 1 1; visual mesh filename=package://jaxon_description/RARM_FINGER1.dae scale=1 1 1
- link RARM_LINK0: geometry collision mesh filename=package://jaxon_description/RARM_LINK0.dae scale=1 1 1; visual mesh filename=package://jaxon_description/RARM_LINK0.dae scale=1 1 1
- link RARM_LINK1: geometry collision mesh filename=package://jaxon_description/RARM_LINK1.dae scale=1 1 1; visual mesh filename=package://jaxon_description/RARM_LINK1.dae scale=1 1 1
- link RARM_LINK2: geometry collision mesh filename=package://jaxon_description/RARM_LINK2.dae scale=1 1 1; visual mesh filename=package://jaxon_description/RARM_LINK2.dae scale=1 1 1
- link RARM_LINK3: geometry collision mesh filename=package://jaxon_description/RARM_LINK3.dae scale=1 1 1; visual mesh filename=package://jaxon_description/RARM_LINK3.dae scale=1 1 1
- link RARM_LINK4: geometry collision mesh filename=package://jaxon_description/RARM_LINK4.dae scale=1 1 1; visual mesh filename=package://jaxon_description/RARM_LINK4.dae scale=1 1 1
- link RARM_LINK5: geometry collision mesh filename=package://jaxon_description/RARM_LINK5.dae scale=1 1 1; visual mesh filename=package://jaxon_description/RARM_LINK5.dae scale=1 1 1
- link RARM_LINK6: geometry collision mesh filename=package://jaxon_description/RARM_LINK6.dae scale=1 1 1; visual mesh filename=package://jaxon_description/RARM_LINK6.dae scale=1 1 1
- link RARM_LINK7: geometry collision mesh filename=package://jaxon_description/RARM_LINK7.dae scale=1 1 1; visual mesh filename=package://jaxon_description/RARM_LINK7.dae scale=1 1 1
- link RLEG_LINK0: geometry collision mesh filename=package://jaxon_description/RLEG_LINK0.dae scale=1 1 1; visual mesh filename=package://jaxon_description/RLEG_LINK0.dae scale=1 1 1
- link RLEG_LINK1: geometry collision mesh filename=package://jaxon_description/RLEG_LINK1.dae scale=1 1 1; visual mesh filename=package://jaxon_description/RLEG_LINK1.dae scale=1 1 1
- link RLEG_LINK2: geometry collision mesh filename=package://jaxon_description/RLEG_LINK2.dae scale=1 1 1; visual mesh filename=package://jaxon_description/RLEG_LINK2.dae scale=1 1 1
- link RLEG_LINK3: geometry collision mesh filename=package://jaxon_description/RLEG_LINK3.dae scale=1 1 1; visual mesh filename=package://jaxon_description/RLEG_LINK3.dae scale=1 1 1
- link RLEG_LINK4: geometry collision mesh filename=package://jaxon_description/RLEG_LINK4.dae scale=1 1 1; visual mesh filename=package://jaxon_description/RLEG_LINK4.dae scale=1 1 1
- link RLEG_LINK5: geometry collision mesh filename=package://jaxon_description/RLEG_LINK5.dae scale=1 1 1; visual mesh filename=package://jaxon_description/RLEG_LINK5.dae scale=1 1 1

Commit message: Fix mesh paths in URDF

File: urdf/jaxon_jvrc.urdf (robot description, URDF)
Before this commit: robot JAXON_JVRC, 39 links, 38 joints
Links:
- link BODY: geometry collision mesh filename=package://jaxon_description/meshes/BODY.dae scale=1 1 1; visual mesh filename=package://jaxon_description/meshes/BODY.dae scale=1 1 1
- link CHEST_LINK0: geometry collision mesh filename=package://jaxon_description/meshes/CHEST_LINK0.dae scale=1 1 1; visual mesh filename=package://jaxon_description/meshes/CHEST_LINK0.dae scale=1 1 1
- link CHEST_LINK1: geometry collision mesh filename=package://jaxon_description/meshes/CHEST_LINK1.dae scale=1 1 1; visual mesh filename=package://jaxon_description/meshes/CHEST_LINK1.dae scale=1 1 1
- link CHEST_LINK2: geometry collision mesh filename=package://jaxon_description/meshes/CHEST_LINK2.dae scale=1 1 1; visual mesh filename=package://jaxon_description/meshes/CHEST_LINK2.dae scale=1 1 1
- link HEAD_LINK0: geometry collision mesh filename=package://jaxon_description/meshes/HEAD_LINK0.dae scale=1 1 1; visual mesh filename=package://jaxon_description/meshes/HEAD_LINK0.dae scale=1 1 1
- link HEAD_LINK1: geometry collision mesh filename=package://jaxon_description/meshes/HEAD_LINK1.dae scale=1 1 1; visual mesh filename=package://jaxon_description/meshes/HEAD_LINK1.dae scale=1 1 1
- link LARM_FINGER0: geometry collision mesh filename=package://jaxon_description/meshes/LARM_FINGER0.dae scale=1 1 1; visual mesh filename=package://jaxon_description/meshes/LARM_FINGER0.dae scale=1 1 1
- link LARM_FINGER1: geometry collision mesh filename=package://jaxon_description/meshes/LARM_FINGER1.dae scale=1 1 1; visual mesh filename=package://jaxon_description/meshes/LARM_FINGER1.dae scale=1 1 1
- link LARM_LINK0: geometry collision mesh filename=package://jaxon_description/meshes/LARM_LINK0.dae scale=1 1 1; visual mesh filename=package://jaxon_description/meshes/LARM_LINK0.dae scale=1 1 1
- link LARM_LINK1: geometry collision mesh filename=package://jaxon_description/meshes/LARM_LINK1.dae scale=1 1 1; visual mesh filename=package://jaxon_description/meshes/LARM_LINK1.dae scale=1 1 1
- link LARM_LINK2: geometry collision mesh filename=package://jaxon_description/meshes/LARM_LINK2.dae scale=1 1 1; visual mesh filename=package://jaxon_description/meshes/LARM_LINK2.dae scale=1 1 1
- link LARM_LINK3: geometry collision mesh filename=package://jaxon_description/meshes/LARM_LINK3.dae scale=1 1 1; visual mesh filename=package://jaxon_description/meshes/LARM_LINK3.dae scale=1 1 1
- link LARM_LINK4: geometry collision mesh filename=package://jaxon_description/meshes/LARM_LINK4.dae scale=1 1 1; visual mesh filename=package://jaxon_description/meshes/LARM_LINK4.dae scale=1 1 1
- link LARM_LINK5: geometry collision mesh filename=package://jaxon_description/meshes/LARM_LINK5.dae scale=1 1 1; visual mesh filename=package://jaxon_description/meshes/LARM_LINK5.dae scale=1 1 1
- link LARM_LINK6: geometry collision mesh filename=package://jaxon_description/meshes/LARM_LINK6.dae scale=1 1 1; visual mesh filename=package://jaxon_description/meshes/LARM_LINK6.dae scale=1 1 1
- link LARM_LINK7: geometry collision mesh filename=package://jaxon_description/meshes/LARM_LINK7.dae scale=1 1 1; visual mesh filename=package://jaxon_description/meshes/LARM_LINK7.dae scale=1 1 1
- link LLEG_LINK0: geometry collision mesh filename=package://jaxon_description/meshes/LLEG_LINK0.dae scale=1 1 1; visual mesh filename=package://jaxon_description/meshes/LLEG_LINK0.dae scale=1 1 1
- link LLEG_LINK1: geometry collision mesh filename=package://jaxon_description/meshes/LLEG_LINK1.dae scale=1 1 1; visual mesh filename=package://jaxon_description/meshes/LLEG_LINK1.dae scale=1 1 1
- link LLEG_LINK2: geometry collision mesh filename=package://jaxon_description/meshes/LLEG_LINK2.dae scale=1 1 1; visual mesh filename=package://jaxon_description/meshes/LLEG_LINK2.dae scale=1 1 1
- link LLEG_LINK3: geometry collision mesh filename=package://jaxon_description/meshes/LLEG_LINK3.dae scale=1 1 1; visual mesh filename=package://jaxon_description/meshes/LLEG_LINK3.dae scale=1 1 1
- link LLEG_LINK4: geometry collision mesh filename=package://jaxon_description/meshes/LLEG_LINK4.dae scale=1 1 1; visual mesh filename=package://jaxon_description/meshes/LLEG_LINK4.dae scale=1 1 1
- link LLEG_LINK5: geometry collision mesh filename=package://jaxon_description/meshes/LLEG_LINK5.dae scale=1 1 1; visual mesh filename=package://jaxon_description/meshes/LLEG_LINK5.dae scale=1 1 1
- link RANGE_LINK: geometry collision mesh filename=package://jaxon_description/meshes/RANGE_LINK.dae scale=1 1 1; visual mesh filename=package://jaxon_description/meshes/RANGE_LINK.dae scale=1 1 1
- link RARM_FINGER0: geometry collision mesh filename=package://jaxon_description/meshes/RARM_FINGER0.dae scale=1 1 1; visual mesh filename=package://jaxon_description/meshes/RARM_FINGER0.dae scale=1 1 1
- link RARM_FINGER1: geometry collision mesh filename=package://jaxon_description/meshes/RARM_FINGER1.dae scale=1 1 1; visual mesh filename=package://jaxon_description/meshes/RARM_FINGER1.dae scale=1 1 1
- link RARM_LINK0: geometry collision mesh filename=package://jaxon_description/meshes/RARM_LINK0.dae scale=1 1 1; visual mesh filename=package://jaxon_description/meshes/RARM_LINK0.dae scale=1 1 1
- link RARM_LINK1: geometry collision mesh filename=package://jaxon_description/meshes/RARM_LINK1.dae scale=1 1 1; visual mesh filename=package://jaxon_description/meshes/RARM_LINK1.dae scale=1 1 1
- link RARM_LINK2: geometry collision mesh filename=package://jaxon_description/meshes/RARM_LINK2.dae scale=1 1 1; visual mesh filename=package://jaxon_description/meshes/RARM_LINK2.dae scale=1 1 1
- link RARM_LINK3: geometry collision mesh filename=package://jaxon_description/meshes/RARM_LINK3.dae scale=1 1 1; visual mesh filename=package://jaxon_description/meshes/RARM_LINK3.dae scale=1 1 1
- link RARM_LINK4: geometry collision mesh filename=package://jaxon_description/meshes/RARM_LINK4.dae scale=1 1 1; visual mesh filename=package://jaxon_description/meshes/RARM_LINK4.dae scale=1 1 1
- link RARM_LINK5: geometry collision mesh filename=package://jaxon_description/meshes/RARM_LINK5.dae scale=1 1 1; visual mesh filename=package://jaxon_description/meshes/RARM_LINK5.dae scale=1 1 1
- link RARM_LINK6: geometry collision mesh filename=package://jaxon_description/meshes/RARM_LINK6.dae scale=1 1 1; visual mesh filename=package://jaxon_description/meshes/RARM_LINK6.dae scale=1 1 1
- link RARM_LINK7: geometry collision mesh filename=package://jaxon_description/meshes/RARM_LINK7.dae scale=1 1 1; visual mesh filename=package://jaxon_description/meshes/RARM_LINK7.dae scale=1 1 1
- link RLEG_LINK0: geometry collision mesh filename=package://jaxon_description/meshes/RLEG_LINK0.dae scale=1 1 1; visual mesh filename=package://jaxon_description/meshes/RLEG_LINK0.dae scale=1 1 1
- link RLEG_LINK1: geometry collision mesh filename=package://jaxon_description/meshes/RLEG_LINK1.dae scale=1 1 1; visual mesh filename=package://jaxon_description/meshes/RLEG_LINK1.dae scale=1 1 1
- link RLEG_LINK2: geometry collision mesh filename=package://jaxon_description/meshes/RLEG_LINK2.dae scale=1 1 1; visual mesh filename=package://jaxon_description/meshes/RLEG_LINK2.dae scale=1 1 1
- link RLEG_LINK3: geometry collision mesh filename=package://jaxon_description/meshes/RLEG_LINK3.dae scale=1 1 1; visual mesh filename=package://jaxon_description/meshes/RLEG_LINK3.dae scale=1 1 1
- link RLEG_LINK4: geometry collision mesh filename=package://jaxon_description/meshes/RLEG_LINK4.dae scale=1 1 1; visual mesh filename=package://jaxon_description/meshes/RLEG_LINK4.dae scale=1 1 1
- link RLEG_LINK5: geometry collision mesh filename=package://jaxon_description/meshes/RLEG_LINK5.dae scale=1 1 1; visual mesh filename=package://jaxon_description/meshes/RLEG_LINK5.dae scale=1 1 1
